File: pcb/ethernetxpansion.kicad_pcb (KiCad board)
At the start: 4 copper layers, 78 x 72.8 mm, 82 parts, among them J1 USB_C_Receptacle_USB2.0_16P, SW1 SW_Push, SW10 SW_Push_45deg, SW11 SW_Push_45deg, SW12 SW_Push_45deg, SW13 SW_Push_45deg, SW14 SW_Push_45deg, SW2 SW_Push, SW3 RotaryEncoder_Switch, SW4 SW_Push_45deg, SW5 SW_Push_45deg, SW6 SW_Push_45deg, SW7 SW_Push_45deg, SW8 SW_Push_45deg, SW9 SW_Push_45deg, U1 MCP1700x-300xxTT, U2 ESP32-C6-MINI-1, U3 RP2040, U4 W25Q16JVSS, Y1 12MHz

Commit message: loads of stuff
Parts:
- removed C17: 0.1uf, Capacitor_SMD:C_0402_1005Metric
- removed D1, D12, D13, D14, D15, D16, D17, D18, D2, D3, D4, D5, D6, D7: WS2812B-2020, LED_SMD:LED_WS2812B-2020_PLCC4_2.0x2.0mm
- removed D10, D11, D19, D20, D21, D22, D29, D30, D31, D32, D8, D9: D_Small, Diode_SMD:D_SOD-323_HandSoldering
- removed D23, D24, D25, D26, D27, D28, D34, D35, D36, D37, D38: LED_SK6812MINI, footprints:MX_SK6812MINI-E
- removed SW1, SW2: SW_Push, Button_Switch_SMD:SW_Push_SPST_NO_Alps_SKRK
- removed SW10, SW11, SW12, SW13, SW14, SW4, SW5, SW6, SW7, SW8, SW9: SW_Push_45deg, Choc:Choc_V1V2_1.00u
- removed SW3: RotaryEncoder_Switch, Rotary_Encoder:RotaryEncoder_Alps_EC11E-Switch_Vertical_H20mm
- removed U2: ESP32-C6-MINI-1, RF_Module:ESP32-C6-MINI-1
- removed U3: RP2040, Package_DFN_QFN:QFN-56-1EP_7x7mm_P0.4mm_EP3.2x3.2mm
- removed U4: W25Q16JVSS, Package_SON:Winbond_USON-8-1EP_3x2mm_P0.5mm_EP0.2x1.6mm
- added J2: RJ45_Hanrun_HR911105A_Horizontal, Connector_RJ:RJ45_Hanrun_HR911105A_Horizontal, F.Cu at (90.2, 53.1)
- added R10: 330R, Resistor_SMD:R_0402_1005Metric, B.Cu at (80.9, 54.4)
- added R11: 49.9, Resistor_SMD:R_0402_1005Metric, B.Cu at (86.5, 69.0)
- added R12: 49.9, Resistor_SMD:R_0402_1005Metric, B.Cu at (86.5, 72.4)
- added R9: 12.4k, Resistor_SMD:R_0402_1005Metric, B.Cu at (89.6, 70.8)
- added REF**: MountingHole_2.2mm_M2, MountingHole:MountingHole_2.2mm_M2, F.Cu at (98.5, 51.1)
- added REF**: MountingHole_2.2mm_M2, MountingHole:MountingHole_2.2mm_M2, F.Cu at (80.2, 70.5)
- C1: value 1uf -> 30pf
- C10, C11, C12, C9: value 100nf -> 100nF
- C13, C14: value 10uf -> 100nF; moved to B.Cu
- C15: value 33pf -> 100nF
- C16: value 33pf -> 1uF
- C2: value 100nf -> 30pf
- C3, C6: value 100nf -> 6.8nF
- C4: value 1uf -> 10nF
- C5: value 100nf -> 4.7uF
- C7: value 100nf -> 22nF
- C8: value 100nf -> 10nF
- J1: value USB_C_Receptacle_USB2.0_16P -> ~; footprint Connector_USB:USB_C_Receptacle_GCT_USB4105-xx-A_16P_TopMnt_Horizontal -> Hackxpansion:Male_Module; moved to F.Cu
- R1: value 10k -> 49.9; footprint Capacitor_SMD:C_0402_1005Metric -> Resistor_SMD:R_0402_1005Metric
- R2: value 5.1k -> 49.9; footprint Capacitor_SMD:C_0402_1005Metric -> Resistor_SMD:R_0402_1005Metric
- R3: value 5.1k -> 10k; footprint Capacitor_SMD:C_0402_1005Metric -> Resistor_SMD:R_0402_1005Metric
- R4: value 27 -> 1M; footprint Capacitor_SMD:C_0402_1005Metric -> Resistor_SMD:R_0402_1005Metric
- R5: value 27 -> 10; footprint Capacitor_SMD:C_0402_1005Metric -> Resistor_SMD:R_0402_1005Metric
- R6: value 1k -> 49.9; footprint Capacitor_SMD:C_0402_1005Metric -> Resistor_SMD:R_0402_1005Metric
- R7: value 10k -> 49.9; footprint Capacitor_SMD:C_0402_1005Metric -> Resistor_SMD:R_0402_1005Metric; moved to B.Cu
- R8: value 1k -> 330R; footprint Capacitor_SMD:C_0402_1005Metric -> Resistor_SMD:R_0402_1005Metric; moved to B.Cu
- U1: value MCP1700x-300xxTT -> W5500; footprint Package_TO_SOT_SMD:SOT-23 -> Package_QFP:LQFP-48_7x7mm_P0.5mm; moved to B.Cu
- Y1: value 12MHz -> 25MHz
- moved R8 74.1 mm to (81.0, 60.6)
- moved R7 68.2 mm to (95.8, 54.4), turned to 180 degrees
- moved U1 61.8 mm to (95.8, 67.5), turned to 45 degrees
- moved C13 59.1 mm to (89.3, 64.2)
- moved C14 56.4 mm to (89.2, 67.2)
- moved R1 50.9 mm to (100.0, 55.5), turned to 0 degrees
- moved Y1 34.9 mm to (98.7, 59.3), turned to 0 degrees
- moved R6 28.5 mm to (92.3, 52.3), turned to 180 degrees
- moved C15 23.1 mm to (90.8, 62.5)
- moved C7 21.8 mm to (95.8, 56.7), turned to 180 degrees
- moved C16 21.0 mm to (88.5, 69.0), turned to 45 degrees
- moved C2 18.7 mm to (100.5, 62.2), turned to -90 degrees
- moved C3 17.8 mm to (86.5, 70.1)
- moved C8 17.4 mm to (86.5, 68.0)
- moved R4 17.1 mm to (98.7, 56.8), turned to 0 degrees
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Connections:
- C1 pad 1: +1V1 -> /XI
- C10 pad 1: +3V3 -> GND
- C10 pad 2: GND -> +3V3
- C11 pad 1: +3V3 -> GND
- C11 pad 2: GND -> +3V3
- C12 pad 1: +3V3 -> GND
- C12 pad 2: GND -> +3V3
- C13 pad 1: +5V -> GND
- C13 pad 2: GND -> +3V3
- C14 pad 1: +3V3 -> GND
- C14 pad 2: GND -> +3V3
- C15 pad 2: /XIN -> +3V3
- C16 pad 2: Net-(C16-Pad2) -> +3V3
- C2 pad 1: +1V1 -> /XO
- C3 pad 1: +1V1 -> /RXP
- C3 pad 2: GND -> /RD+
- C4 pad 1: +3V3 -> GND
- C4 pad 2: GND -> Net-(U1-1V2O)
- C5 pad 1: +3V3 -> GND
- C5 pad 2: GND -> Net-(U1-TOCAP)
- C6 pad 1: +3V3 -> /RXN
- C6 pad 2: GND -> /RD-
- C7 pad 1: +3V3 -> GND
- C7 pad 2: GND -> Net-(J2-TCT)
- C8 pad 1: +3V3 -> GND
- C8 pad 2: GND -> Net-(J2-RCT)
- C9 pad 1: +3V3 -> GND
- C9 pad 2: GND -> +3V3
- R1 pad 1: Net-(U2-EN) -> +3V3
- R1 pad 2: +3V3 -> Net-(J1-MD0)
- R2 pad 1: Net-(J1-CC1) -> +3V3
- R2 pad 2: GND -> Net-(J1-MD1)
- R3 pad 1: Net-(J1-CC2) -> +3V3
- R3 pad 2: GND -> /RST
- R4 pad 1: /D+ -> /XI
- R4 pad 2: Net-(U3-USB_DP) -> /XO
- R5 pad 1: /D- -> +3V3
- R5 pad 2: Net-(U3-USB_DM) -> Net-(J2-TCT)
- R6 pad 1: Net-(C16-Pad2) -> +3V3
- R6 pad 2: /XOUT -> /TXP
- R7 pad 1: /QSPI_SS -> +3V3
- R7 pad 2: +3V3 -> /TXN
- R8 pad 2: /QSPI_SS -> /LINKLED
- U1 pad 1: GND -> /TXN
- U1 pad 2: +3V3 -> /TXP
- U1 pad 3: +5V -> GND
- Y1 pad 1: Net-(C16-Pad2) -> /XI
- Y1 pad 3: /XIN -> /XO
Routing:
- net /c4: track 88.8 -> 0.00 mm, vias 1 -> 0
- net +3V3: track 57.6 -> 145.0 mm, vias 0 -> 4
- net /r3: track 86.8 -> 0.00 mm
- net /r2: track 84.7 -> 0.00 mm
- net /r1: track 74.1 -> 0.00 mm
- net /c3: track 66.5 -> 0.00 mm, vias 1 -> 0
- net /c1: track 61.5 -> 0.00 mm, vias 1 -> 0
- net /c2: track 51.5 -> 0.00 mm, vias 1 -> 0
- net Net-(D3-DOUT): track 34.2 -> 0.00 mm
- net /D+: track 31.0 -> 0.00 mm
- net /D-: track 29.8 -> 0.00 mm
- net /TXP: track 0.00 -> 28.0 mm, vias 0 -> 2
- net /ACTLED: track 0.00 -> 27.6 mm, vias 0 -> 2
- net /RD-: track 0.00 -> 25.3 mm, vias 0 -> 2
- net /TXN: track 0.00 -> 23.1 mm, vias 0 -> 1
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- added copper zone on F.Cu, net GND
- added copper zone on In2.Cu, net GND
- removed copper zone on In2.Cu, net +5V
Other:
- board size 78 x 72.8 mm -> 32 x 25.5 mm
