File: pcb/ethernetxpansion.kicad_sch (KiCad schematic)
At the start: 24 parts, among them J3 RJ45_Hanrun_HR911105A_Horizon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, U1 W5500, Y2 25MHz

Commit message: loads of stuff
Parts:
- added C10, C11, C12, C13, C14, C15, C9: 100nF, Capacitor_SMD:C_0402_1005Metric, symbol Device:C_Small
- added C16: 1uF, Capacitor_SMD:C_0402_1005Metric, symbol Device:C_Small
- C1, C2: footprint Package_SO:SOIC-8_3.9x4.9mm_P1.27mm -> Capacitor_SMD:C_0402_1005Metric
- C3: renamed from C4; footprint (none) -> Capacitor_SMD:C_0402_1005Metric
- C4: renamed from C7; footprint (none) -> Capacitor_SMD:C_0402_1005Metric
- C5: renamed from C8; footprint (none) -> Capacitor_SMD:C_0402_1005Metric
- C6: renamed from C3; footprint (none) -> Capacitor_SMD:C_0402_1005Metric
- C7: renamed from C5; footprint (none) -> Capacitor_SMD:C_0402_1005Metric
- C8: renamed from C6; footprint (none) -> Capacitor_SMD:C_0402_1005Metric
- R1: renamed from R12; value 49.9 -> 1k1; footprint Resistor_THT:R_Array_SIP4 -> Resistor_SMD:R_0402_1005Metric
- R10: renamed from R2; footprint Connector_RJ:RJ45_Hanrun_HR911105A_Horizontal -> Resistor_SMD:R_0402_1005Metric
- R11: renamed from R7; footprint Resistor_THT:R_Array_SIP4 -> Resistor_SMD:R_0402_1005Metric
- R12: renamed from R8; footprint Resistor_THT:R_Array_SIP4 -> Resistor_SMD:R_0402_1005Metric
- R2: renamed from R11; value 49.9 -> 1k8; footprint Resistor_THT:R_Array_SIP4 -> Resistor_SMD:R_0402_1005Metric
- R3: footprint Connector_RJ:RJ45_Hanrun_HR911105A_Horizontal -> Resistor_SMD:R_0402_1005Metric
- R4: renamed from R10; footprint Resistor_THT:R_Array_SIP4 -> Resistor_SMD:R_0402_1005Metric
- R5: renamed from R6; footprint Resistor_THT:R_Array_SIP4 -> Resistor_SMD:R_0402_1005Metric
- R6: renamed from R5; footprint Resistor_THT:R_Array_SIP4 -> Resistor_SMD:R_0402_1005Metric
- R7: renamed from R4; footprint Resistor_THT:R_Array_SIP4 -> Resistor_SMD:R_0402_1005Metric
- R8: renamed from R1; footprint Connector_RJ:RJ45_Hanrun_HR911105A_Horizontal -> Resistor_SMD:R_0402_1005Metric
- R9: footprint Resistor_THT:R_Array_SIP4 -> Resistor_SMD:R_0402_1005Metric
- Y1: renamed from Y2; footprint (none) -> Crystal:Crystal_SMD_3225-4Pin_3.2x2.5mm
- renumbered J3 to J2
Connections:
- net +3V3: now also C10.2, C11.2, C12.2, C13.2, C14.2, C15.2, C16.2, C9.2
- net GND: now also C10.1, C11.1, C12.1, C13.1, C14.1, C15.1, C16.1, C9.1
- net RD+: now reaches C3.2, J2.3 (RD+)
- net RD-: now reaches C6.2, J2.6 (RD-)
Other:
- moved on the sheet: C1, C2, C3, C4, C5, C6, C7, C8, J1, J2, R1, R10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
